File: circuit/keyflogger.kicad_pcb (KiCad board)
At the start: 2 copper layers, 45 x 19 mm, 20 parts, among them J1 USB_A, J2 USB_B_Micro, J3 Conn_PIC_ICSP_ICD, J4 Conn_PIC_ICSP_ICD, Q1 2N7002, Q2 2N7002, U1 PIC16F1454-IP, U2 PIC16F1454-IP

Commit message: circuit: Update LED labels to reflect functional symmetry
The firmware is identical on each side, and the device may be used in
whichever orientation is more physically convenient.  Update the LED
labels to reflect this symmetry.

Signed-off-by: Michael Brown <mbrown@fensystems.co.uk>
Other:
- board text added: "A"
- board text added: "B"
- board text removed: "GADGET"
- board text removed: "KB/MOUSE"

Commit message: circuit: Add fiducial markers
Signed-off-by: Michael Brown <mbrown@fensystems.co.uk>
Parts:
- added F1: Fiducial, Fiducial:Fiducial_1mm_Mask2mm, F.Cu at (142.9, 96.3)
- added F2: Fiducial, Fiducial:Fiducial_1mm_Mask2mm, F.Cu at (148.7, 112.0)
- added F3: Fiducial, Fiducial:Fiducial_1mm_Mask2mm, F.Cu at (175.8, 112.0)

Commit message: circuit: Add bill of materials
Signed-off-by: Michael Brown <mbrown@fensystems.co.uk>
Parts:
- D1, D2: value LED -> Red 2mA
